Commit message: polygons were added

File: urdf_models/models/polygons/2_poly.xacro (robot description, xacro)
@@ -12,7 +12,7 @@
   limitations under the License.
 -->
-<robot name="3_poly" xmlns:xacro="http://ros.org/wiki/xacro">
-  <xacro:property name="mesh_file" value="package://urdf_models/models/stone/3D_models_3.dae" />
-  <xacro:property name="mass" value="1.0" />
+<robot name="2_poly" xmlns:xacro="http://ros.org/wiki/xacro">
+  <xacro:property name="mesh_file" value="package://urdf_models/models/polygons/2_poly.stl" />
+  <xacro:property name="mass" value="0.5" />
   <link name="base_link"></link>
   <joint name="base_joint" type="fixed">
@@ -24,9 +24,9 @@
       <inertial>
         <mass value="${mass}" />  <!-- [kg] -->
-        <origin xyz="0 0 0.12" />
-        <inertia ixx="1" ixy="0.0" ixz="0.0"
-                 iyy="1" iyz="0.0"
-                 izz="1" />
-      </inertial>
+        <origin xyz=" 0.00 0.0 0.0" />
+        <inertia ixx="0.000001" ixy="0.0" 		ixz="0.0"
+                			      iyy="0.000001"  iyz="0.0"
+                 								    izz="0.000001" />
+        </inertial>
       <visual>
         <origin xyz="0 0 0" rpy="0 0 0" />

File: urdf_models/models/polygons/3_poly.xacro (robot description, xacro)
@@ -12,7 +12,7 @@
   limitations under the License.
 -->
-<robot name="1_poly" xmlns:xacro="http://ros.org/wiki/xacro">
-  <xacro:property name="mesh_file" value="package://urdf_models/models/stone/3D_models_1.dae" />
-  <xacro:property name="mass" value="1.0" />
+<robot name="3_poly" xmlns:xacro="http://ros.org/wiki/xacro">
+  <xacro:property name="mesh_file" value="package://urdf_models/models/polygons/3_poly.stl" />
+  <xacro:property name="mass" value="0.5" />
   <link name="base_link"></link>
   <joint name="base_joint" type="fixed">
@@ -24,8 +24,8 @@
       <inertial>
         <mass value="${mass}" />  <!-- [kg] -->
-        <origin xyz="0 0 0.12" />
-        <inertia ixx="1" ixy="0.0" ixz="0.0"
-                 iyy="1" iyz="0.0"
-                 izz="1" />
+        <origin xyz="-0.004250 -0.001861  0.004301" />
+        <inertia ixx="0.00000056" ixy="0.0" 		ixz="0.0"
+                			    iyy="0.00000076"  iyz="0.0"
+                 								izz="0.00000083" />
       </inertial>
       <visual>
@@ -45,3 +45,7 @@
       </collision>
     </link>
+   <gazebo reference="$base_link_inertia">
+        <mu1>1.1</mu1>
+        <mu2>1.1</mu2>
+   </gazebo>
 </robot>

File: urdf_models/models/polygons/4_poly.xacro (robot description, xacro)
@@ -12,7 +12,7 @@
   limitations under the License.
 -->
-<robot name="2_poly" xmlns:xacro="http://ros.org/wiki/xacro">
-  <xacro:property name="mesh_file" value="package://urdf_models/models/stone/3D_models_2.dae" />
-  <xacro:property name="mass" value="1.0" />
+<robot name="3_poly" xmlns:xacro="http://ros.org/wiki/xacro">
+  <xacro:property name="mesh_file" value="package://urdf_models/models/polygons/4_poly.stl" />
+  <xacro:property name="mass" value="0.3" />
   <link name="base_link"></link>
   <joint name="base_joint" type="fixed">
@@ -24,8 +24,8 @@
       <inertial>
         <mass value="${mass}" />  <!-- [kg] -->
-        <origin xyz="0 0 0.12" />
-        <inertia ixx="1" ixy="0.0" ixz="0.0"
-                 iyy="1" iyz="0.0"
-                 izz="1" />
+        <origin xyz="0.0 0.0 0.0" />
+        <inertia ixx="0.000001" ixy="0.0" 		ixz="0.0"
+                			    iyy="0.000001"  iyz="0.0"
+                 								izz="0.000001" />
       </inertial>
       <visual>
@@ -45,3 +45,7 @@
       </collision>
     </link>
+   <gazebo reference="$base_link_inertia">
+        <mu1>1.1</mu1>
+        <mu2>1.1</mu2>
+   </gazebo>
 </robot>
