Commit message: fixed inertia tensors

File: urdf_models/models/polygons/1_poly.xacro (robot description, xacro)
@@ -24,8 +24,8 @@
       <inertial>
         <mass value="${mass}" />  <!-- [kg] -->
-        <origin xyz=" -0.095090 0.139665  0.037921" />
-        <inertia ixx="0.000001" ixy="0.0" 		ixz="0.0"
-                			    iyy="0.000001"  iyz="0.0"
-                 								izz="0.000001" />
+        <origin xyz="0.172716e-02 0.036106e-02 0.106380e-02" />
+        <inertia ixx="0.063821e-05" ixy="0.0" 		ixz="0.0"
+                			    iyy="0.105141e-05"  iyz="0.0"
+                 								izz="0.110947e-05" />
       </inertial>
       <visual>

File: urdf_models/models/polygons/2_poly.xacro (robot description, xacro)
@@ -24,8 +24,8 @@
       <inertial>
         <mass value="${mass}" />  <!-- [kg] -->
-        <origin xyz=" 0.00 0.0 0.0" />
-        <inertia ixx="0.000001" ixy="0.0" 		ixz="0.0"
-                			      iyy="0.000001"  iyz="0.0"
-                 								    izz="0.000001" />
+        <origin xyz=" 0.048762e-02 0.004925e-02 0.025797e-02" />
+        <inertia ixx="0.033551e-05" ixy="0.0" 		ixz="0.0"
+                			      iyy="0.039115e-05"  iyz="0.0"
+                 								    izz="0.036632e-05" />
         </inertial>
       <visual>

File: urdf_models/models/polygons/3_poly.xacro (robot description, xacro)
@@ -24,8 +24,8 @@
       <inertial>
         <mass value="${mass}" />  <!-- [kg] -->
-        <origin xyz="-0.004250 -0.001861  0.004301" />
-        <inertia ixx="0.00000056" ixy="0.0" 		ixz="0.0"
-                			    iyy="0.00000076"  iyz="0.0"
-                 								izz="0.00000083" />
+        <origin xyz="-0.042501e-02 -0.0018606e-02  0.0043009e-02" />
+        <inertia ixx="0.005698e-05" ixy="0.0" 		ixz="0.0"
+                			    iyy="0.007699e-05"  iyz="0.0"
+                 								izz="0.008392e-05" />
       </inertial>
       <visual>

File: urdf_models/models/polygons/4_poly.xacro (robot description, xacro)
@@ -24,8 +24,8 @@
       <inertial>
         <mass value="${mass}" />  <!-- [kg] -->
-        <origin xyz="0.0 0.0 0.0" />
-        <inertia ixx="0.000001" ixy="0.0" 		ixz="0.0"
-                			    iyy="0.000001"  iyz="0.0"
-                 								izz="0.000001" />
+        <origin xyz="-0.005615e-02 -0.005404e-02  -0.060523e-02 " />
+        <inertia ixx="0.007005e-05" ixy="0.0" 		ixz="0.0"
+                			    iyy="0.004923e-05"  iyz="0.0"
+                 								izz="0.008620e-05" />
       </inertial>
       <visual>

File: urdf_models/models/polygons/5_poly.xacro (robot description, xacro)
@@ -24,8 +24,8 @@
       <inertial>
         <mass value="${mass}" />  <!-- [kg] -->
-        <origin xyz="0.0 0.0 0.0" />
-        <inertia ixx="0.000001" ixy="0.0" 		ixz="0.0"
-                			    iyy="0.000001"  iyz="0.0"
-                 								izz="0.000001" />
+        <origin xyz="0.008764e-02 0.010792e-02 -0.014634e-02" />
+        <inertia ixx="0.002472e-05" ixy="0.0" 		ixz="0.0"
+                			    iyy="0.002012e-05"  iyz="0.0"
+                 								izz="0.003289e-05" />
       </inertial>
       <visual>

Commit message: for demo

File: urdf_models/models/polygons/1_poly.xacro (robot description, xacro)
@@ -24,8 +24,8 @@
       <inertial>
         <mass value="${mass}" />  <!-- [kg] -->
-        <origin xyz="0.172716e-02 0.036106e-02 0.106380e-02" />
-        <inertia ixx="0.063821e-05" ixy="0.0" 		ixz="0.0"
-                			    iyy="0.105141e-05"  iyz="0.0"
-                 								izz="0.110947e-05" />
+        <origin xyz="0.172716e-01 0.036106e-01 0.106380e-01" />
+        <inertia ixx="0.063821e-02" ixy="0.0" 		ixz="0.0"
+                			    iyy="0.105141e-02"  iyz="0.0"
+                 								izz="0.110947e-02" />
       </inertial>
       <visual>

File: urdf_models/models/polygons/3_poly.xacro (robot description, xacro)
@@ -24,8 +24,8 @@
       <inertial>
         <mass value="${mass}" />  <!-- [kg] -->
-        <origin xyz="-0.042501e-02 -0.0018606e-02  0.0043009e-02" />
-        <inertia ixx="0.005698e-05" ixy="0.0" 		ixz="0.0"
-                			    iyy="0.007699e-05"  iyz="0.0"
-                 								izz="0.008392e-05" />
+        <origin xyz="-0.042501e-01 -0.0018606e-01  0.0043009e-01" />
+        <inertia ixx="0.005698e-02" ixy="0.0" 		ixz="0.0"
+                			    iyy="0.007699e-02"  iyz="0.0"
+                 								izz="0.008392e-02" />
       </inertial>
       <visual>
@@ -48,4 +48,6 @@
         <mu1>1.1</mu1>
         <mu2>1.1</mu2>
+        <kp>1000000.0</kp>
+        <kd>1.0</kd>
    </gazebo>
 </robot>

File: urdf_models/models/polygons/4_poly.xacro (robot description, xacro)
@@ -13,6 +13,6 @@
 -->
 <robot name="3_poly" xmlns:xacro="http://ros.org/wiki/xacro">
-  <xacro:property name="mesh_file" value="package://urdf_models/models/polygons/4_poly.stl" />
-  <xacro:property name="mass" value="0.3" />
+  <xacro:property name="mesh_file" value="package://urdf_models/models/polygons/4_poly_2.stl" />
+  <xacro:property name="mass" value="0.1" />
   <link name="base_link"></link>
   <joint name="base_joint" type="fixed">
@@ -24,8 +24,8 @@
       <inertial>
         <mass value="${mass}" />  <!-- [kg] -->
-        <origin xyz="-0.005615e-02 -0.005404e-02  -0.060523e-02 " />
-        <inertia ixx="0.007005e-05" ixy="0.0" 		ixz="0.0"
-                			    iyy="0.004923e-05"  iyz="0.0"
-                 								izz="0.008620e-05" />
+        <origin xyz="-0.010158e-01 -0.025367e-01  -0.008778e-01 " />
+        <inertia ixx="0.003829e-02" ixy="-0.000181e-02" 	ixz="0.000153e-02"
+                			    iyy="0.003572e-02"  iyz="0.0000063e-02"
+                 								izz="0.004654e-02" />
       </inertial>
       <visual>
@@ -43,9 +43,21 @@
           <mesh filename="${mesh_file}" scale="1 1 1" />
         </geometry>
+        <surface>
+          	<friction>
+          		<ode>
+            		<mu>1.2</mu>
+            		<mu2>1.2</mu2>
+          		</ode>
+        	</friction>
+            <bounce>
+              <restitution_coefficient>10.0</restitution_coefficient>
+            </bounce>
+            <contact>
+              <ode>
+                <max_vel>10</max_vel>
+              </ode>
+            </contact>
+        </surface>
       </collision>
     </link>
-   <gazebo reference="$base_link_inertia">
-        <mu1>1.1</mu1>
-        <mu2>1.1</mu2>
-   </gazebo>
 </robot>

File: urdf_models/models/polygons/5_poly.xacro (robot description, xacro)
@@ -14,5 +14,5 @@
 <robot name="3_poly" xmlns:xacro="http://ros.org/wiki/xacro">
   <xacro:property name="mesh_file" value="package://urdf_models/models/polygons/5_poly.stl" />
-  <xacro:property name="mass" value="0.3" />
+  <xacro:property name="mass" value="1.2" />
   <link name="base_link"></link>
   <joint name="base_joint" type="fixed">
@@ -24,8 +24,8 @@
       <inertial>
         <mass value="${mass}" />  <!-- [kg] -->
-        <origin xyz="0.008764e-02 0.010792e-02 -0.014634e-02" />
-        <inertia ixx="0.002472e-05" ixy="0.0" 		ixz="0.0"
-                			    iyy="0.002012e-05"  iyz="0.0"
-                 								izz="0.003289e-05" />
+        <origin xyz="0.008764e-01 0.010792e-01 -0.014634e-01" />
+        <inertia ixx="0.002472e-02" ixy="0.0" 		ixz="0.0"
+                			    iyy="0.002012e-02"  iyz="0.0"
+                 								izz="0.003289e-02" />
       </inertial>
       <visual>
@@ -34,7 +34,4 @@
           <mesh filename="${mesh_file}" scale="1 1 1" />
         </geometry>
-	<material name="blue">
-	  <color rgba="0 0 .8 1"/>
-	</material>
       </visual>
       <collision>
@@ -43,9 +40,21 @@
           <mesh filename="${mesh_file}" scale="1 1 1" />
         </geometry>
+        <surface>
+          	<friction>
+          		<ode>
+            		<mu>1.2</mu>
+            		<mu2>1.2</mu2>
+          		</ode>
+        	</friction>
+            <bounce>
+              <restitution_coefficient>10.0</restitution_coefficient>
+            </bounce>
+            <contact>
+              <ode>
+                <max_vel>10</max_vel>
+              </ode>
+            </contact>
+        </surface>
       </collision>
     </link>
-   <gazebo reference="$base_link_inertia">
-        <mu1>1.1</mu1>
-        <mu2>1.1</mu2>
-   </gazebo>
 </robot>

Commit message: coefficient settings

File: urdf_models/models/polygons/1_poly.xacro (robot description, xacro)
@@ -34,7 +34,7 @@
           <mesh filename="${mesh_file}" scale="1 1 1" />
         </geometry>
-	<material name="blue">
-	  <color rgba="0 0 .8 1"/>
-	</material>
+		<material name="Gray">
+	 	 <color rgba="0.8 0.8 0.8 1"/>
+		</material>
       </visual>
       <collision>
@@ -43,9 +43,29 @@
           <mesh filename="${mesh_file}" scale="1 1 1" />
         </geometry>
+        <surface>
+          <bounce>
+            <restitution_coefficient> 0.1 </restitution_coefficient>
+          </bounce>
+        </surface>
       </collision>
-    </link>
-   <gazebo reference="$base_link_inertia">
-        <mu1>1.1</mu1>
-        <mu2>1.1</mu2>
-   </gazebo>
+  </link>
+  <gazebo reference="base_link">
+      <mu1 value="2.1"/>
+      <mu2 value="1.1"/>
+      <kp  value="5000000.0" />
+      <kd  value="1.0" />
+      <surface>
+        <contact>
+          <ode>
+            <max_vel>0.5</max_vel>
+            <min_depth>0.001</min_depth>
+          </ode>
+        </contact>
+      </surface>
+      <fdir1 value="1 0 0"/>
+      <material name="Gray">
+	    <color rgba="0.8 0.8 0.8 1"/>
+	  </material>
+      <turnGravityOff>false</turnGravityOff>
+  </gazebo>
 </robot>

File: urdf_models/models/polygons/2_poly.xacro (robot description, xacro)
@@ -44,4 +44,4 @@
         </geometry>
       </collision>
-    </link>
+  </link>
 </robot>

File: urdf_models/models/polygons/5_poly.xacro (robot description, xacro)
@@ -25,7 +25,7 @@
         <mass value="${mass}" />  <!-- [kg] -->
         <origin xyz="0.008764e-01 0.010792e-01 -0.014634e-01" />
-        <inertia ixx="0.002472e-02" ixy="0.0" 		ixz="0.0"
-                			    iyy="0.002012e-02"  iyz="0.0"
-                 								izz="0.003289e-02" />
+        <inertia ixx="0.002472e-02" ixy="0.0" 			ixz="0.0"
+                			    	iyy="0.002012e-02"  iyz="0.0"
+                 										izz="0.003289e-02" />
       </inertial>
       <visual>
@@ -48,5 +48,5 @@
         	</friction>
             <bounce>
-              <restitution_coefficient>10.0</restitution_coefficient>
+              <restitution_coefficient>0.1</restitution_coefficient>
             </bounce>
             <contact>

Commit message: parameters are working on gazebo

File: urdf_models/models/polygons/1_poly.xacro (robot description, xacro)
@@ -43,25 +43,26 @@
           <mesh filename="${mesh_file}" scale="1 1 1" />
         </geometry>
-        <surface>
-          <bounce>
-            <restitution_coefficient> 0.1 </restitution_coefficient>
-          </bounce>
-        </surface>
       </collision>
   </link>
   <gazebo reference="base_link">
-      <mu1 value="2.1"/>
+      <mu1 value="1.2"/>
       <mu2 value="1.1"/>
       <kp  value="5000000.0" />
       <kd  value="1.0" />
-      <surface>
-        <contact>
-          <ode>
-            <max_vel>0.5</max_vel>
-            <min_depth>0.001</min_depth>
-          </ode>
-        </contact>
-      </surface>
       <fdir1 value="1 0 0"/>
+      <collision>
+	        <surface>
+	          <bounce>
+	            <restitution_coefficient> 0.1 </restitution_coefficient>
+	            <threshold>0.</threshold>
+	          </bounce>
+		      <contact>
+		          <ode>
+		            <max_vel>0.1</max_vel>
+		            <min_depth>0.001</min_depth>
+		          </ode>
+		      </contact>
+	        </surface>
+	   </collision>
       <material name="Gray">
 	    <color rgba="0.8 0.8 0.8 1"/>

File: urdf_models/models/polygons/2_poly.xacro (robot description, xacro)
@@ -45,3 +45,28 @@
       </collision>
   </link>
+  <gazebo reference="base_link">
+      <mu1 value="1.2"/>
+      <mu2 value="1.1"/>
+      <kp  value="5000000.0" />
+      <kd  value="1.0" />
+      <fdir1 value="1 0 0"/>
+      <collision>
+	        <surface>
+	          <bounce>
+	            <restitution_coefficient> 0.1 </restitution_coefficient>
+	            <threshold>0.</threshold>
+	          </bounce>
+		      <contact>
+		          <ode>
+		            <max_vel>0.1</max_vel>
+		            <min_depth>0.001</min_depth>
+		          </ode>
+		      </contact>
+	        </surface>
+	   </collision>
+      <material name="Gray">
+	    <color rgba="0.8 0.8 0.8 1"/>
+	  </material>
+      <turnGravityOff>false</turnGravityOff>
+  </gazebo>
 </robot>

File: urdf_models/models/polygons/3_poly.xacro (robot description, xacro)
@@ -14,5 +14,5 @@
 <robot name="3_poly" xmlns:xacro="http://ros.org/wiki/xacro">
   <xacro:property name="mesh_file" value="package://urdf_models/models/polygons/3_poly.stl" />
-  <xacro:property name="mass" value="0.5" />
+  <xacro:property name="mass" value="1.0" />
   <link name="base_link"></link>
   <joint name="base_joint" type="fixed">
@@ -34,6 +34,6 @@
           <mesh filename="${mesh_file}" scale="1 1 1" />
         </geometry>
-	<material name="blue">
-	  <color rgba="0 0 .8 1"/>
+	<material name="Gray">
+	  <color rgba="0.8 0.8 0.8 1"/>
 	</material>
       </visual>
@@ -45,9 +45,28 @@
       </collision>
     </link>
-   <gazebo reference="$base_link_inertia">
-        <mu1>1.1</mu1>
-        <mu2>1.1</mu2>
-        <kp>1000000.0</kp>
-        <kd>1.0</kd>
-   </gazebo>
+    <gazebo reference="base_link">
+      <mu1 value="1.2"/>
+      <mu2 value="1.1"/>
+      <kp  value="5000000.0" />
+      <kd  value="1.0" />
+      <fdir1 value="1 0 0"/>
+      <collision>
+	        <surface>
+	          <bounce>
+	            <restitution_coefficient> 0.1 </restitution_coefficient>
+	            <threshold>0.</threshold>
+	          </bounce>
+		      <contact>
+		          <ode>
+		            <max_vel>0.1</max_vel>
+		            <min_depth>0.001</min_depth>
+		          </ode>
+		      </contact>
+	        </surface>
+	   </collision>
+      <material name="Gray">
+	    <color rgba="0.8 0.8 0.8 1"/>
+	  </material>
+      <turnGravityOff>false</turnGravityOff>
+    </gazebo>
 </robot>

File: urdf_models/models/polygons/4_poly.xacro (robot description, xacro)
@@ -12,10 +12,10 @@
   limitations under the License.
 -->
-<robot name="3_poly" xmlns:xacro="http://ros.org/wiki/xacro">
-  <xacro:property name="mesh_file" value="package://urdf_models/models/polygons/4_poly_2.stl" />
-  <xacro:property name="mass" value="0.1" />
+<robot name="4_poly" xmlns:xacro="http://ros.org/wiki/xacro">
+  <xacro:property name="mesh_file" value="package://urdf_models/models/polygons/4_poly_3.stl" />
+  <xacro:property name="mass" value="1.0" />
   <link name="base_link"></link>
   <joint name="base_joint" type="fixed">
-    <origin xyz="0 0 0" rpy="0 0 0" />
+    <origin xyz="0 0 0" rpy="-2.21 -1.47 0.215" />
     <parent link="base_link" />
     <child link="base_link_inertia" />
@@ -24,8 +24,8 @@
       <inertial>
         <mass value="${mass}" />  <!-- [kg] -->
-        <origin xyz="-0.010158e-01 -0.025367e-01  -0.008778e-01 " />
-        <inertia ixx="0.003829e-02" ixy="-0.000181e-02" 	ixz="0.000153e-02"
-                			    iyy="0.003572e-02"  iyz="0.0000063e-02"
-                 								izz="0.004654e-02" />
+        <origin xyz="0.022361e-01 -0.016301e-01  -0.007616e-01 " />
+        <inertia ixx="0.003908e-02" ixy="-0.0" 			ixz="0."
+                			    	iyy="0.003465e-02"  iyz="0.0"
+                 										izz="0.004682e-02" />
       </inertial>
       <visual>
@@ -34,7 +34,7 @@
           <mesh filename="${mesh_file}" scale="1 1 1" />
         </geometry>
-	<material name="blue">
-	  <color rgba="0 0 .8 1"/>
-	</material>
+		<material name="Gray">
+	 	 <color rgba="0.8 0.8 0.8 1"/>
+		</material>
       </visual>
       <collision>
@@ -43,21 +43,30 @@
           <mesh filename="${mesh_file}" scale="1 1 1" />
         </geometry>
-        <surface>
-          	<friction>
-          		<ode>
-            		<mu>1.2</mu>
-            		<mu2>1.2</mu2>
-          		</ode>
-        	</friction>
-            <bounce>
-              <restitution_coefficient>10.0</restitution_coefficient>
-            </bounce>
-            <contact>
-              <ode>
-                <max_vel>10</max_vel>
-              </ode>
-            </contact>
-        </surface>
       </collision>
     </link>
+    <gazebo reference="base_link">
+      <mu1 value="1.2"/>
+      <mu2 value="1.1"/>
+      <kp  value="5000000.0" />
+      <kd  value="1.0" />
+      <fdir1 value="1 0 0"/>
+      <collision>
+	        <surface>
+	          <bounce>
+	            <restitution_coefficient> 0.1 </restitution_coefficient>
+	            <threshold>0.</threshold>
+	          </bounce>
+		      <contact>
+		          <ode>
+		            <max_vel>0.1</max_vel>
+		            <min_depth>0.001</min_depth>
+		          </ode>
+		      </contact>
+	        </surface>
+	   </collision>
+      <material name="Gray">
+	    <color rgba="0.8 0.8 0.8 1"/>
+	  </material>
+      <turnGravityOff>false</turnGravityOff>
+    </gazebo>
 </robot>

File: urdf_models/models/polygons/5_poly.xacro (robot description, xacro)
@@ -12,7 +12,7 @@
   limitations under the License.
 -->
-<robot name="3_poly" xmlns:xacro="http://ros.org/wiki/xacro">
+<robot name="5_poly" xmlns:xacro="http://ros.org/wiki/xacro">
   <xacro:property name="mesh_file" value="package://urdf_models/models/polygons/5_poly.stl" />
-  <xacro:property name="mass" value="1.2" />
+  <xacro:property name="mass" value="1.0" />
   <link name="base_link"></link>
   <joint name="base_joint" type="fixed">
@@ -25,7 +25,7 @@
         <mass value="${mass}" />  <!-- [kg] -->
         <origin xyz="0.008764e-01 0.010792e-01 -0.014634e-01" />
-        <inertia ixx="0.002472e-02" ixy="0.0" 			ixz="0.0"
-                			    	iyy="0.002012e-02"  iyz="0.0"
-                 										izz="0.003289e-02" />
+        <inertia ixx="0.002472e-01" ixy="0.0" 			ixz="0.0"
+                			    	iyy="0.002012e-01"  iyz="0.0"
+                 										izz="0.003289e-01" />
       </inertial>
       <visual>
@@ -40,21 +40,30 @@
           <mesh filename="${mesh_file}" scale="1 1 1" />
         </geometry>
-        <surface>
-          	<friction>
-          		<ode>
-            		<mu>1.2</mu>
-            		<mu2>1.2</mu2>
-          		</ode>
-        	</friction>
-            <bounce>
-              <restitution_coefficient>0.1</restitution_coefficient>
-            </bounce>
-            <contact>
-              <ode>
-                <max_vel>10</max_vel>
-              </ode>
-            </contact>
-        </surface>
       </collision>
     </link>
+  <gazebo reference="base_link">
+      <mu1 value="1.2"/>
+      <mu2 value="1.1"/>
+      <kp  value="5000000.0" />
+      <kd  value="1.0" />
+      <fdir1 value="1 0 0"/>
+      <collision>
+	        <surface>
+	          <bounce>
+	            <restitution_coefficient> 0.1 </restitution_coefficient>
+	            <threshold>0.</threshold>
+	          </bounce>
+		      <contact>
+		          <ode>
+		            <max_vel>0.1</max_vel>
+		            <min_depth>0.001</min_depth>
+		          </ode>
+		      </contact>
+	        </surface>
+	   </collision>
+      <material name="Gray">
+	    <color rgba="0.8 0.8 0.8 1"/>
+	  </material>
+      <turnGravityOff>false</turnGravityOff>
+  </gazebo>
 </robot>
