Commit message: I modified Poly1's initial pose and inertia.

File: urdf_models/models/1_poly/1_poly.xacro (robot description, xacro)
@@ -17,5 +17,5 @@
   <link name="base_link"></link>
   <joint name="base_joint" type="fixed">
-    <origin xyz="0 0 0" rpy="0 0 0" />
+    <origin xyz="0 0 0" rpy="0 -0.4 0" />
     <parent link="base_link" />
     <child link="base_link_inertia" />
