Commit message: file structure was changed

File: urdf_models/models/stone/urdf/stone.xacro (robot description, xacro)
@@ -12,6 +12,6 @@
   limitations under the License.
 -->
-<robot name="2_poly" xmlns:xacro="http://ros.org/wiki/xacro">
-  <xacro:property name="mesh_file" value="package://urdf_models/models/stone/3D_models_2.dae" />
+<robot name="stone" xmlns:xacro="http://ros.org/wiki/xacro">
+  <xacro:property name="mesh_file" value="package://urdf_models/models/stone/mesh/stone.dae" />
   <xacro:property name="mass" value="1.0" />
   <link name="base_link"></link>
@@ -34,7 +34,4 @@
           <mesh filename="${mesh_file}" scale="1 1 1" />
         </geometry>
-	<material name="blue">
-	  <color rgba="0 0 .8 1"/>
-	</material>
       </visual>
       <collision>

File: urdf_models/models/stone_1/urdf/stone_1.xacro (robot description, xacro)
@@ -12,6 +12,6 @@
   limitations under the License.
 -->
-<robot name="2_poly" xmlns:xacro="http://ros.org/wiki/xacro">
-  <xacro:property name="mesh_file" value="package://urdf_models/models/stone/3D_models_1.dae" />
+<robot name="stone_1" xmlns:xacro="http://ros.org/wiki/xacro">
+<xacro:property name="mesh_file" value="package://urdf_models/models/stone_1/mesh/stone_1.stl" />
   <xacro:property name="mass" value="1.0" />
   <link name="base_link"></link>
@@ -22,11 +22,11 @@
   </joint>
   <link name="base_link_inertia">
-      <inertial>
-        <mass value="${mass}" />  <!-- [kg] -->
-        <origin xyz="0 0 0.12" />
-        <inertia ixx="1" ixy="0.0" ixz="0.0"
-                 iyy="1" iyz="0.0"
-                 izz="1" />
-      </inertial>
+  <inertial>
+    <mass value="${mass}" />  <!-- [kg] -->
+    <origin xyz="-0.0029634 0.0067405 0.0403623" />
+    <inertia ixx="0.023458e-02" ixy="-0.002390e-02" ixz="0.004260e-02"
+                                iyy="0.030342e-02"  iyz="0.002545e-02"
+                                                    izz="0.033413e-02" />
+   </inertial>
       <visual>
         <origin xyz="0 0 0" rpy="0 0 0" />
@@ -34,7 +34,4 @@
           <mesh filename="${mesh_file}" scale="1 1 1" />
         </geometry>
-	<material name="blue">
-	  <color rgba="0 0 .8 1"/>
-	</material>
       </visual>
       <collision>
@@ -45,3 +42,28 @@
       </collision>
     </link>
+    <gazebo reference="base_link">
+        <mu1 value="2.2"/>
+        <mu2 value="1.1"/>
+        <kp  value="5000000.0" />
+        <kd  value="1.0" />
+        <fdir1 value="1 0 0"/>
+        <collision>
+            <surface>
+              <bounce>
+                <restitution_coefficient> 0.1 </restitution_coefficient>
+                <threshold>0.</threshold>
+              </bounce>
+            <contact>
+                <ode>
+                  <max_vel>0.1</max_vel>
+                  <min_depth>0.001</min_depth>
+                </ode>
+            </contact>
+            </surface>
+       </collision>
+        <material name="Gray">
+        <color rgba="0.8 0.8 0.8 1"/>
+      </material>
+        <turnGravityOff>false</turnGravityOff>
+    </gazebo>
 </robot>

File: urdf_models/models/stone_2/urdf/stone_2.xacro (robot description, xacro)
@@ -12,6 +12,6 @@
   limitations under the License.
 -->
-<robot name="stone" xmlns:xacro="http://ros.org/wiki/xacro">
-  <xacro:property name="mesh_file" value="package://urdf_models/models/stone/stone.dae" />
+<robot name="stone_2" xmlns:xacro="http://ros.org/wiki/xacro">
+  <xacro:property name="mesh_file" value="package://urdf_models/models/stone_2/mesh/stone_2.stl" />
   <xacro:property name="mass" value="1.0" />
   <link name="base_link"></link>
@@ -24,8 +24,8 @@
       <inertial>
         <mass value="${mass}" />  <!-- [kg] -->
-        <origin xyz="0 0 0.12" />
-        <inertia ixx="1" ixy="0.0" ixz="0.0"
-                 iyy="1" iyz="0.0"
-                 izz="1" />
+        <origin xyz="0.172716e-01 0.036106e-01 0.106380e-01" />
+        <inertia ixx="0.063821e-02" ixy="0.0" 		ixz="0.0"
+                			    iyy="0.105141e-02"  iyz="0.0"
+                 								izz="0.110947e-02" />
       </inertial>
       <visual>
@@ -34,4 +34,7 @@
           <mesh filename="${mesh_file}" scale="1 1 1" />
         </geometry>
+		<material name="Gray">
+	 	 <color rgba="0.8 0.8 0.8 1"/>
+		</material>
       </visual>
       <collision>
@@ -41,4 +44,29 @@
         </geometry>
       </collision>
-    </link>
+  </link>
+  <gazebo reference="base_link">
+      <mu1 value="1.2"/>
+      <mu2 value="1.1"/>
+      <kp  value="5000000.0" />
+      <kd  value="1.0" />
+      <fdir1 value="1 0 0"/>
+      <collision>
+	        <surface>
+	          <bounce>
+	            <restitution_coefficient> 0.1 </restitution_coefficient>
+	            <threshold>0.</threshold>
+	          </bounce>
+		      <contact>
+		          <ode>
+		            <max_vel>0.1</max_vel>
+		            <min_depth>0.001</min_depth>
+		          </ode>
+		      </contact>
+	        </surface>
+	   </collision>
+      <material name="Gray">
+	    <color rgba="0.8 0.8 0.8 1"/>
+	  </material>
+      <turnGravityOff>false</turnGravityOff>
+  </gazebo>
 </robot>

File: urdf_models/models/template/urdf/template.xacro (robot description, xacro)
@@ -12,6 +12,6 @@
   limitations under the License.
 -->
-<robot name="2_poly" xmlns:xacro="http://ros.org/wiki/xacro">
-  <xacro:property name="mesh_file" value="package://urdf_models/models/stone/3D_models_1.dae" />
+<robot name="template" xmlns:xacro="http://ros.org/wiki/xacro">
+  <xacro:property name="mesh_file" value="package://urdf_models/models/mesh/template.stl" />
   <xacro:property name="mass" value="1.0" />
   <link name="base_link"></link>
@@ -24,8 +24,8 @@
       <inertial>
         <mass value="${mass}" />  <!-- [kg] -->
-        <origin xyz="0 0 0.12" />
-        <inertia ixx="1" ixy="0.0" ixz="0.0"
-                 iyy="1" iyz="0.0"
-                 izz="1" />
+        <origin xyz="0.172716e-01 0.036106e-01 0.106380e-01" />
+        <inertia ixx="0.063821e-02" ixy="0.0" 		ixz="0.0"
+                			    iyy="0.105141e-02"  iyz="0.0"
+                 								izz="0.110947e-02" />
       </inertial>
       <visual>
@@ -34,7 +34,7 @@
           <mesh filename="${mesh_file}" scale="1 1 1" />
         </geometry>
-	<material name="blue">
-	  <color rgba="0 0 .8 1"/>
-	</material>
+		<material name="Gray">
+	 	 <color rgba="0.8 0.8 0.8 1"/>
+		</material>
       </visual>
       <collision>
@@ -44,4 +44,29 @@
         </geometry>
       </collision>
-    </link>
+  </link>
+  <gazebo reference="base_link">
+      <mu1 value="1.2"/>
+      <mu2 value="1.1"/>
+      <kp  value="5000000.0" />
+      <kd  value="1.0" />
+      <fdir1 value="1 0 0"/>
+      <collision>
+	        <surface>
+	          <bounce>
+	            <restitution_coefficient> 0.1 </restitution_coefficient>
+	            <threshold>0.</threshold>
+	          </bounce>
+		      <contact>
+		          <ode>
+		            <max_vel>0.1</max_vel>
+		            <min_depth>0.001</min_depth>
+		          </ode>
+		      </contact>
+	        </surface>
+	   </collision>
+      <material name="Gray">
+	    <color rgba="0.8 0.8 0.8 1"/>
+	  </material>
+      <turnGravityOff>false</turnGravityOff>
+  </gazebo>
 </robot>
