Commit message: cleaned other files.

File: urdf_models/models/stone_highres/urdf/stone.xacro (robot description, xacro)
@@ -12,7 +12,7 @@
   limitations under the License.
 -->
-<robot name="2_poly" xmlns:xacro="http://ros.org/wiki/xacro">
-  <xacro:property name="mesh_file" value="package://urdf_models/meshes/2_stone.dae" />
-  <xacro:property name="mass" value="1" />
+<robot name="stone_highres" xmlns:xacro="http://ros.org/wiki/xacro">
+  <xacro:property name="mesh_file" value="package://urdf_models/models/stone/mesh/stone.dae" />
+  <xacro:property name="mass" value="1.0" />
   <link name="base_link"></link>
   <joint name="base_joint" type="fixed">
@@ -24,9 +24,9 @@
       <inertial>
         <mass value="${mass}" />  <!-- [kg] -->
-        <origin xyz=" -0.002491 -0.000222 -0.004263" />
-        <inertia ixx="0.065740e-02" ixy="0.001483e-02" 		ixz="-0.000435e-02"
-                			      	      iyy="0.021578e-02"  	iyz="0.000101e-02"
-                 								    		                  izz="0.0720994e-02" />
-        </inertial>
+        <origin xyz="0 0 0.12" />
+        <inertia ixx="1" ixy="0.0" ixz="0.0"
+                 iyy="1" iyz="0.0"
+                 izz="1" />
+      </inertial>
       <visual>
         <origin xyz="0 0 0" rpy="0 0 0" />
@@ -41,29 +41,4 @@
         </geometry>
       </collision>
-  </link>
-  <gazebo reference="base_link">
-      <mu1 value="1.2"/>
-      <mu2 value="1.1"/>
-      <kp  value="5000000.0" />
-      <kd  value="1.0" />
-      <fdir1 value="1 0 0"/>
-      <collision>
-	        <surface>
-	          <bounce>
-	            <restitution_coefficient> 0.1 </restitution_coefficient>
-	            <threshold>0.</threshold>
-	          </bounce>
-		      <contact>
-		          <ode>
-		            <max_vel>0.1</max_vel>
-		            <min_depth>0.001</min_depth>
-		          </ode>
-		      </contact>
-	        </surface>
-	   </collision>
-      <material name="Gray">
-	    <color rgba="0.8 0.8 0.8 1"/>
-	  </material>
-      <turnGravityOff>false</turnGravityOff>
-  </gazebo>
+    </link>
 </robot>
