Commit message: fixed the structure

File: urdf_models/models/1_poly/urdf/1_poly.xacro (robot description, xacro)
@@ -12,6 +12,6 @@
   limitations under the License.
 -->
-<robot name="3_poly" xmlns:xacro="http://ros.org/wiki/xacro">
-  <xacro:property name="mesh_file" value="package://urdf_models/models/polygons/3_poly.stl" />
+<robot name="1_poly" xmlns:xacro="http://ros.org/wiki/xacro">
+  <xacro:property name="mesh_file" value="package://urdf_models/models/1_poly/mesh/1_poly.stl" />
   <xacro:property name="mass" value="1.0" />
   <link name="base_link"></link>
@@ -24,8 +24,8 @@
       <inertial>
         <mass value="${mass}" />  <!-- [kg] -->
-        <origin xyz="-0.042501e-01 -0.0018606e-01  0.0043009e-01" />
-        <inertia ixx="0.005698e-02" ixy="0.0" 		ixz="0.0"
-                			    iyy="0.007699e-02"  iyz="0.0"
-                 								izz="0.008392e-02" />
+        <origin xyz="0.172716e-01 0.036106e-01 0.106380e-01" />
+        <inertia ixx="0.063821e-02" ixy="0.0" 		ixz="0.0"
+                			    iyy="0.105141e-02"  iyz="0.0"
+                 								izz="0.110947e-02" />
       </inertial>
       <visual>
@@ -34,7 +34,7 @@
           <mesh filename="${mesh_file}" scale="1 1 1" />
         </geometry>
-	<material name="Gray">
-	  <color rgba="0.8 0.8 0.8 1"/>
-	</material>
+		<material name="Gray">
+	 	 <color rgba="0.8 0.8 0.8 1"/>
+		</material>
       </visual>
       <collision>
@@ -44,6 +44,6 @@
         </geometry>
       </collision>
-    </link>
-    <gazebo reference="base_link">
+  </link>
+  <gazebo reference="base_link">
       <mu1 value="1.2"/>
       <mu2 value="1.1"/>
@@ -69,4 +69,4 @@
 	  </material>
       <turnGravityOff>false</turnGravityOff>
-    </gazebo>
+  </gazebo>
 </robot>

File: urdf_models/models/2_poly/urdf/2_poly.xacro (robot description, xacro)
@@ -12,7 +12,7 @@
   limitations under the License.
 -->
-<robot name="5_poly" xmlns:xacro="http://ros.org/wiki/xacro">
-  <xacro:property name="mesh_file" value="package://urdf_models/models/polygons/5_poly.stl" />
-  <xacro:property name="mass" value="1.0" />
+<robot name="2_poly" xmlns:xacro="http://ros.org/wiki/xacro">
+  <xacro:property name="mesh_file" value="package://urdf_models/models/2_poly/mesh/2_poly.stl" />
+  <xacro:property name="mass" value="1" />
   <link name="base_link"></link>
   <joint name="base_joint" type="fixed">
@@ -24,9 +24,9 @@
       <inertial>
         <mass value="${mass}" />  <!-- [kg] -->
-        <origin xyz="0.008764e-01 0.010792e-01 -0.014634e-01" />
-        <inertia ixx="0.002472e-01" ixy="0.0" 			ixz="0.0"
-                			    	iyy="0.002012e-01"  iyz="0.0"
-                 										izz="0.003289e-01" />
-      </inertial>
+        <origin xyz=" -0.160056e-1  0.049179e-1 0.080512e-1" />
+        <inertia ixx="0.034550e-02" ixy="0.000148e-02" 		ixz="0.001628e-02"
+                			      	iyy="0.038334e-02"  	iyz="0.001259e-02"
+                 								    		izz="0.036534e-02" />
+        </inertial>
       <visual>
         <origin xyz="0 0 0" rpy="0 0 0" />
@@ -34,4 +34,7 @@
           <mesh filename="${mesh_file}" scale="1 1 1" />
         </geometry>
+	<material name="blue">
+	  <color rgba="0 0 .8 1"/>
+	</material>
       </visual>
       <collision>
@@ -41,5 +44,5 @@
         </geometry>
       </collision>
-    </link>
+  </link>
   <gazebo reference="base_link">
       <mu1 value="1.2"/>

File: urdf_models/models/3_poly/urdf/3_poly.xacro (robot description, xacro)
@@ -12,7 +12,7 @@
   limitations under the License.
 -->
-<robot name="2_poly" xmlns:xacro="http://ros.org/wiki/xacro">
-  <xacro:property name="mesh_file" value="package://urdf_models/models/polygons/2_poly_config_2.dae" />
-  <xacro:property name="mass" value="1" />
+<robot name="3_poly" xmlns:xacro="http://ros.org/wiki/xacro">
+  <xacro:property name="mesh_file" value="package://urdf_models/models/3_poly/mesh/3_poly.stl" />
+  <xacro:property name="mass" value="1.0" />
   <link name="base_link"></link>
   <joint name="base_joint" type="fixed">
@@ -24,9 +24,9 @@
       <inertial>
         <mass value="${mass}" />  <!-- [kg] -->
-        <origin xyz=" -0.160056e-1  0.049179e-1 0.080512e-1" />
-        <inertia ixx="0.034550e-02" ixy="0.000148e-02" 		ixz="0.001628e-02"
-                			      	iyy="0.038334e-02"  	iyz="0.001259e-02"
-                 								    		izz="0.036534e-02" />
-        </inertial>
+        <origin xyz="-0.042501e-01 -0.0018606e-01  0.0043009e-01" />
+        <inertia ixx="0.005698e-02" ixy="0.0" 		ixz="0.0"
+                			    iyy="0.007699e-02"  iyz="0.0"
+                 								izz="0.008392e-02" />
+      </inertial>
       <visual>
         <origin xyz="0 0 0" rpy="0 0 0" />
@@ -34,6 +34,6 @@
           <mesh filename="${mesh_file}" scale="1 1 1" />
         </geometry>
-	<material name="blue">
-	  <color rgba="0 0 .8 1"/>
+	<material name="Gray">
+	  <color rgba="0.8 0.8 0.8 1"/>
 	</material>
       </visual>
@@ -44,6 +44,6 @@
         </geometry>
       </collision>
-  </link>
-  <gazebo reference="base_link">
+    </link>
+    <gazebo reference="base_link">
       <mu1 value="1.2"/>
       <mu2 value="1.1"/>
@@ -69,4 +69,4 @@
 	  </material>
       <turnGravityOff>false</turnGravityOff>
-  </gazebo>
+    </gazebo>
 </robot>

File: urdf_models/models/4_poly/urdf/4_poly.xacro (robot description, xacro)
@@ -13,5 +13,5 @@
 -->
 <robot name="4_poly" xmlns:xacro="http://ros.org/wiki/xacro">
-  <xacro:property name="mesh_file" value="package://urdf_models/models/polygons/4_poly_3.stl" />
+  <xacro:property name="mesh_file" value="package://urdf_models/models/4_poly/mesh/4_poly_3.stl" />
   <xacro:property name="mass" value="1.0" />
   <link name="base_link"></link>

File: urdf_models/models/5_poly/urdf/5_poly.xacro (robot description, xacro)
@@ -12,6 +12,6 @@
   limitations under the License.
 -->
-<robot name="1_poly" xmlns:xacro="http://ros.org/wiki/xacro">
-  <xacro:property name="mesh_file" value="package://urdf_models/models/polygons/1_poly.stl" />
+<robot name="5_poly" xmlns:xacro="http://ros.org/wiki/xacro">
+  <xacro:property name="mesh_file" value="package://urdf_models/models/5_poly/mesh/5_poly.stl" />
   <xacro:property name="mass" value="1.0" />
   <link name="base_link"></link>
@@ -24,8 +24,8 @@
       <inertial>
         <mass value="${mass}" />  <!-- [kg] -->
-        <origin xyz="0.172716e-01 0.036106e-01 0.106380e-01" />
-        <inertia ixx="0.063821e-02" ixy="0.0" 		ixz="0.0"
-                			    iyy="0.105141e-02"  iyz="0.0"
-                 								izz="0.110947e-02" />
+        <origin xyz="0.008764e-01 0.010792e-01 -0.014634e-01" />
+        <inertia ixx="0.002472e-01" ixy="0.0" 			ixz="0.0"
+                			    	iyy="0.002012e-01"  iyz="0.0"
+                 										izz="0.003289e-01" />
       </inertial>
       <visual>
@@ -34,7 +34,4 @@
           <mesh filename="${mesh_file}" scale="1 1 1" />
         </geometry>
-		<material name="Gray">
-	 	 <color rgba="0.8 0.8 0.8 1"/>
-		</material>
       </visual>
       <collision>
@@ -44,5 +41,5 @@
         </geometry>
       </collision>
-  </link>
+    </link>
   <gazebo reference="base_link">
       <mu1 value="1.2"/>

Commit message: fixed folder structure and launch files

File: urdf_models/models/1_poly/urdf/1_poly.xacro (robot description, xacro)
@@ -12,10 +12,10 @@
   limitations under the License.
 -->
-<robot name="4_poly" xmlns:xacro="http://ros.org/wiki/xacro">
-  <xacro:property name="mesh_file" value="package://urdf_models/models/polygons/4_poly_3.stl" />
+<robot name="1_poly" xmlns:xacro="http://ros.org/wiki/xacro">
+  <xacro:property name="mesh_file" value="package://urdf_models/models/1_poly/mesh/1_poly.stl" />
   <xacro:property name="mass" value="1.0" />
   <link name="base_link"></link>
   <joint name="base_joint" type="fixed">
-    <origin xyz="0 0 0" rpy="-2.21 -1.47 0.215" />
+    <origin xyz="0 0 0" rpy="0 0 0" />
     <parent link="base_link" />
     <child link="base_link_inertia" />
@@ -24,8 +24,8 @@
       <inertial>
         <mass value="${mass}" />  <!-- [kg] -->
-        <origin xyz="0.022361e-01 -0.016301e-01  -0.007616e-01 " />
-        <inertia ixx="0.003908e-02" ixy="-0.0" 			ixz="0."
-                			    	iyy="0.003465e-02"  iyz="0.0"
-                 										izz="0.004682e-02" />
+        <origin xyz="0.172716e-01 0.036106e-01 0.106380e-01" />
+        <inertia ixx="0.063821e-02" ixy="0.0" 		ixz="0.0"
+                			    iyy="0.105141e-02"  iyz="0.0"
+                 								izz="0.110947e-02" />
       </inertial>
       <visual>
@@ -44,6 +44,6 @@
         </geometry>
       </collision>
-    </link>
-    <gazebo reference="base_link">
+  </link>
+  <gazebo reference="base_link">
       <mu1 value="1.2"/>
       <mu2 value="1.1"/>
@@ -69,4 +69,4 @@
 	  </material>
       <turnGravityOff>false</turnGravityOff>
-    </gazebo>
+  </gazebo>
 </robot>

File: urdf_models/models/4_poly/urdf/4_poly.xacro (robot description, xacro)
@@ -12,10 +12,10 @@
   limitations under the License.
 -->
-<robot name="stone_highres" xmlns:xacro="http://ros.org/wiki/xacro">
-  <xacro:property name="mesh_file" value="package://urdf_models/models/stone/mesh/stone.dae" />
+<robot name="4_poly" xmlns:xacro="http://ros.org/wiki/xacro">
+  <xacro:property name="mesh_file" value="package://urdf_models/models/4_poly/mesh/4_poly_3.stl" />
   <xacro:property name="mass" value="1.0" />
   <link name="base_link"></link>
   <joint name="base_joint" type="fixed">
-    <origin xyz="0 0 0" rpy="0 0 0" />
+    <origin xyz="0 0 0" rpy="-2.21 -1.47 0.215" />
     <parent link="base_link" />
     <child link="base_link_inertia" />
@@ -24,8 +24,8 @@
       <inertial>
         <mass value="${mass}" />  <!-- [kg] -->
-        <origin xyz="0 0 0.12" />
-        <inertia ixx="1" ixy="0.0" ixz="0.0"
-                 iyy="1" iyz="0.0"
-                 izz="1" />
+        <origin xyz="0.022361e-01 -0.016301e-01  -0.007616e-01 " />
+        <inertia ixx="0.003908e-02" ixy="-0.0" 			ixz="0."
+                			    	iyy="0.003465e-02"  iyz="0.0"
+                 										izz="0.004682e-02" />
       </inertial>
       <visual>
@@ -34,4 +34,7 @@
           <mesh filename="${mesh_file}" scale="1 1 1" />
         </geometry>
+		<material name="Gray">
+	 	 <color rgba="0.8 0.8 0.8 1"/>
+		</material>
       </visual>
       <collision>
@@ -42,3 +45,28 @@
       </collision>
     </link>
+    <gazebo reference="base_link">
+      <mu1 value="1.2"/>
+      <mu2 value="1.1"/>
+      <kp  value="5000000.0" />
+      <kd  value="1.0" />
+      <fdir1 value="1 0 0"/>
+      <collision>
+	        <surface>
+	          <bounce>
+	            <restitution_coefficient> 0.1 </restitution_coefficient>
+	            <threshold>0.</threshold>
+	          </bounce>
+		      <contact>
+		          <ode>
+		            <max_vel>0.1</max_vel>
+		            <min_depth>0.001</min_depth>
+		          </ode>
+		      </contact>
+	        </surface>
+	   </collision>
+      <material name="Gray">
+	    <color rgba="0.8 0.8 0.8 1"/>
+	  </material>
+      <turnGravityOff>false</turnGravityOff>
+    </gazebo>
 </robot>
