Commit message: different file was called from stone_2 mesh. It's fixed now.

File: urdf_models/models/stone_2/urdf/stone_2.xacro (robot description, xacro)
@@ -13,5 +13,5 @@
 -->
 <robot name="stone_2" xmlns:xacro="http://ros.org/wiki/xacro">
-  <xacro:property name="mesh_file" value="package://urdf_models/models/stone_2/mesh/stone_2.stl" />
+  <xacro:property name="mesh_file" value="package://urdf_models/models/stone_2/mesh/stone_2_2.stl" />
   <xacro:property name="mass" value="1.0" />
   <link name="base_link"></link>

Commit message: added new stone models from laser scans

File: urdf_models/models/stone_2/urdf/stone_2.xacro (robot description, xacro)
@@ -13,5 +13,5 @@
 -->
 <robot name="stone_2" xmlns:xacro="http://ros.org/wiki/xacro">
-  <xacro:property name="mesh_file" value="package://urdf_models/models/stone_2/mesh/stone_2_2.stl" />
+  <xacro:property name="mesh_file" value="package://urdf_models/models/stone_2/mesh/stone_2.stl" />
   <xacro:property name="mass" value="1.0" />
   <link name="base_link"></link>

File: urdf_models/models/stone_4/urdf/stone_4.xacro (robot description, xacro)
@@ -12,6 +12,6 @@
   limitations under the License.
 -->
-<robot name="stone_1" xmlns:xacro="http://ros.org/wiki/xacro">
-  <xacro:property name="mesh_file" value="package://urdf_models/models/stone_1/mesh/stone_1.stl" />
+<robot name="stone_4" xmlns:xacro="http://ros.org/wiki/xacro">
+  <xacro:property name="mesh_file" value="package://urdf_models/models/stone_4/mesh/stone_4.stl" />
   <xacro:property name="mass" value="1.0" />
   <link name="base_link"></link>

File: urdf_models/models/stone_5/urdf/stone_5.xacro (robot description, xacro)
@@ -12,6 +12,6 @@
   limitations under the License.
 -->
-<robot name="stone_1" xmlns:xacro="http://ros.org/wiki/xacro">
-  <xacro:property name="mesh_file" value="package://urdf_models/models/stone_1/mesh/stone_1.stl" />
+<robot name="stone_5" xmlns:xacro="http://ros.org/wiki/xacro">
+<xacro:property name="mesh_file" value="package://urdf_models/models/stone_5/mesh/stone_5.stl" />
   <xacro:property name="mass" value="1.0" />
   <link name="base_link"></link>

File: urdf_models/models/stone_6/urdf/stone_6.xacro (robot description, xacro)
@@ -12,6 +12,6 @@
   limitations under the License.
 -->
-<robot name="stone_1" xmlns:xacro="http://ros.org/wiki/xacro">
-  <xacro:property name="mesh_file" value="package://urdf_models/models/stone_1/mesh/stone_1.stl" />
+<robot name="stone_6" xmlns:xacro="http://ros.org/wiki/xacro">
+<xacro:property name="mesh_file" value="package://urdf_models/models/stone_6/mesh/stone_6.stl" />
   <xacro:property name="mass" value="1.0" />
   <link name="base_link"></link>

Commit message: Some formatting.

File: urdf_models/models/stone_2/urdf/stone_2.xacro (robot description, xacro)
@@ -46,27 +46,27 @@
   </link>
   <gazebo reference="base_link">
-        <mu1 value="0.1"/>
-        <mu2 value="0.1"/>
-      <kp  value="5000000.0" />
-      <kd  value="1.0" />
-      <fdir1 value="1 0 0"/>
-      <collision>
-	      <surface>
-	          <bounce>
-	            <restitution_coefficient> 0.0 </restitution_coefficient>
-	            <threshold>0.</threshold>
-	          </bounce>
-		        <contact>
-		          <ode>
-		            <max_vel>10</max_vel>
-		            <min_depth>0.001</min_depth>
-		          </ode>
-		        </contact>
-	      </surface>
-	   </collision>
-      <material name="Gray">
-	    <color rgba="0.8 0.8 0.8 1"/>
-	  </material>
-      <turnGravityOff>false</turnGravityOff>
+    <mu1 value="0.1"/>
+    <mu2 value="0.1"/>
+    <kp  value="5000000.0" />
+    <kd  value="1.0" />
+    <fdir1 value="1 0 0"/>
+    <collision>
+      <surface>
+        <bounce>
+          <restitution_coefficient> 0.0 </restitution_coefficient>
+          <threshold>0.</threshold>
+        </bounce>
+  	    <contact>
+  	      <ode>
+  	        <max_vel>10</max_vel>
+  	        <min_depth>0.001</min_depth>
+  	      </ode>
+  	    </contact>
+      </surface>
+    </collision>
+    <material name="Gray">
+      <color rgba="0.8 0.8 0.8 1"/>
+    </material>
+    <turnGravityOff>false</turnGravityOff>
   </gazebo>
 </robot>

File: urdf_models/models/stone_3/urdf/stone_3.xacro (robot description, xacro)
@@ -46,27 +46,27 @@
   </link>
   <gazebo reference="base_link">
-        <mu1 value="0.1"/>
-        <mu2 value="0.1"/>
-      <kp  value="5000000.0" />
-      <kd  value="1.0" />
-      <fdir1 value="1 0 0"/>
-      <collision>
-	        <surface>
-	          <bounce>
-	            <restitution_coefficient> 10 </restitution_coefficient>
-	            <threshold>0.</threshold>
-	          </bounce>
-		      <contact>
-		          <ode>
-		            <max_vel>0.1</max_vel>
-		            <min_depth>0.001</min_depth>
-		          </ode>
-		      </contact>
-	        </surface>
-	   </collision>
-      <material name="Gray">
-	    <color rgba="0.8 0.8 0.8 1"/>
-	  </material>
-      <turnGravityOff>false</turnGravityOff>
+    <mu1 value="0.1"/>
+    <mu2 value="0.1"/>
+    <kp  value="5000000.0" />
+    <kd  value="1.0" />
+    <fdir1 value="1 0 0"/>
+    <collision>
+      <surface>
+        <bounce>
+          <restitution_coefficient> 0.1 </restitution_coefficient>
+          <threshold>0.</threshold>
+        </bounce>
+  	    <contact>
+  	      <ode>
+  	        <max_vel>10.0</max_vel>
+  	        <min_depth>0.001</min_depth>
+  	      </ode>
+  	    </contact>
+      </surface>
+    </collision>
+    <material name="Gray">
+      <color rgba="0.8 0.8 0.8 1"/>
+    </material>
+    <turnGravityOff>false</turnGravityOff>
   </gazebo>
 </robot>
