Commit message: fixed xacro files for the stones for demo.

File: urdf_models/models/stone_1/urdf/stone_1.xacro (robot description, xacro)
@@ -24,8 +24,8 @@
   <inertial>
     <mass value="${mass}" />  <!-- [kg] -->
-    <origin xyz="-0.0029634 0.0067405 0.0403623" />
-    <inertia ixx="0.023458e-02" ixy="-0.002390e-02" ixz="0.004260e-02"
-                                iyy="0.030342e-02"  iyz="0.002545e-02"
-                                                    izz="0.033413e-02" />
+    <origin xyz="-0.0000142 0.0000139 0.0000031" />
+    <inertia ixx="0.008166e-02" ixy="-0.003668e-02" ixz="-0.000031e-02"
+                                iyy="0.020183e-02"  iyz="0.000657e-02"
+                                                    izz="0.024189e-02" />
    </inertial>
       <visual>

File: urdf_models/models/stone_2/urdf/stone_2.xacro (robot description, xacro)
@@ -24,8 +24,8 @@
       <inertial>
         <mass value="${mass}" />  <!-- [kg] -->
-        <origin xyz="0.179580e-01 0.281355e-01 0.480871e-01" />
-        <inertia ixx="0.239644e-02"  ixy="-0.027213e-02"  ixz="-0.001755e-02"
-                			               iyy="0.084688e-02"  iyz="-0.004446e-02"
-                 								                         izz="0.267884e-02" />
+        <origin xyz="-0.000322e-1 -0.000145e-1 -0.000170e-1" />
+        <inertia ixx="0.019941e-02"  ixy="0.004477e-02"  ixz="-0.002525e-02"
+                			               iyy="0.030632e-02"  iyz="-0.002664e-02"
+                 								                         izz="0.040836e-02" />
       </inertial>
       <visual>

File: urdf_models/models/stone_3/urdf/stone_3.xacro (robot description, xacro)
@@ -24,17 +24,17 @@
       <inertial>
         <mass value="${mass}" />  <!-- [kg] -->
-        <origin xyz="-0.276797e-01 0.786830e-01 0.457372e-01" />
-       <inertia ixx="0.008036e-02"  ixy="0.000346e-02"  ixz="-0.000609e-02"
-                                    iyy="0.013250e-02"  iyz="0.000933e-02"
-                                                        izz="0.013387e-02" />
+        <origin xyz=" 0.000056e-1 0.000026e-1 0.000159e-1" />
+       <inertia ixx="0.005936e-02"  ixy="-0.001673e-02"  ixz="0.00102e-02"
+                                    iyy="0.008784e-02"  iyz="0.001319e-02"
+                                                        izz="0.010867e-02" />
       </inertial>
       <visual>
         <origin xyz="0 0 0" rpy="0 0 0" />
-        <geometry>
-          <mesh filename="${mesh_file}" scale="1 1 1" />
-        </geometry>
-		<material name="Gray">
-	 	 <color rgba="0.8 0.8 0.8 1"/>
-		</material>
+          <geometry>
+            <mesh filename="${mesh_file}" scale="1 1 1" />
+          </geometry>
+		      <material name="Gray">
+	 	        <color rgba="0.8 0.8 0.8 1"/>
+		      </material>
       </visual>
       <collision>

File: urdf_models/models/stone_4/urdf/stone_4.xacro (robot description, xacro)
@@ -22,24 +22,24 @@
   </joint>
   <link name="base_link_inertia">
-  <inertial>
-    <mass value="${mass}" />  <!-- [kg] -->
-    <origin xyz="-0.0029634 0.0067405 0.0403623" />
-    <inertia ixx="0.023458e-02" ixy="-0.002390e-02" ixz="0.004260e-02"
-                                iyy="0.030342e-02"  iyz="0.002545e-02"
-                                                    izz="0.033413e-02" />
-   </inertial>
-      <visual>
-        <origin xyz="0 0 0" rpy="0 0 0" />
-        <geometry>
-          <mesh filename="${mesh_file}" scale="1 1 1" />
-        </geometry>
-      </visual>
-      <collision>
-        <origin xyz="0 0 0" rpy="0 0 0" />
-        <geometry>
-          <mesh filename="${mesh_file}" scale="1 1 1" />
-        </geometry>
-      </collision>
-    </link>
+    <inertial>
+      <mass value="${mass}" />  <!-- [kg] -->
+      <origin xyz="-0.000019e-1 0.000016e-1 -0.000054e-1" />
+      <inertia ixx="0.007451e-02" ixy="0.002706e-02" ixz="0.000231e-02"
+                                iyy="0.012215e-02"  iyz="-0.001176e-02"
+                                                    izz="0.013797e-02" />
+    </inertial>
+    <visual>
+      <origin xyz="0 0 0" rpy="0 0 0" />
+      <geometry>
+        <mesh filename="${mesh_file}" scale="1 1 1" />
+      </geometry>
+    </visual>
+    <collision>
+      <origin xyz="0 0 0" rpy="0 0 0" />
+      <geometry>
+        <mesh filename="${mesh_file}" scale="1 1 1" />
+      </geometry>
+    </collision>
+  </link>
     <gazebo reference="base_link">
         <mu1 value="2.2"/>

File: urdf_models/models/stone_5/urdf/stone_5.xacro (robot description, xacro)
@@ -24,8 +24,8 @@
   <inertial>
     <mass value="${mass}" />  <!-- [kg] -->
-    <origin xyz="-0.0029634 0.0067405 0.0403623" />
-    <inertia ixx="0.023458e-02" ixy="-0.002390e-02" ixz="0.004260e-02"
-                                iyy="0.030342e-02"  iyz="0.002545e-02"
-                                                    izz="0.033413e-02" />
+    <origin xyz="0.000209e-1 0.000129e-1 0.000045e-1" />
+    <inertia ixx="0.005520e-02" ixy="-0.001326e-02" ixz="0.000610e-02"
+                                iyy="0.006123e-02"  iyz="-0.001059e-02"
+                                                    izz="0.009342e-02" />
    </inertial>
       <visual>

File: urdf_models/models/stone_6/urdf/stone_6.xacro (robot description, xacro)
@@ -24,8 +24,8 @@
   <inertial>
     <mass value="${mass}" />  <!-- [kg] -->
-    <origin xyz="-0.0029634 0.0067405 0.0403623" />
-    <inertia ixx="0.023458e-02" ixy="-0.002390e-02" ixz="0.004260e-02"
-                                iyy="0.030342e-02"  iyz="0.002545e-02"
-                                                    izz="0.033413e-02" />
+    <origin xyz=" -0.021062e-1 -0.000296e-1 0.000037e-1" />
+    <inertia ixx="0.012356e-02" ixy="0.002844e-02" ixz="-0.000649e-02"
+                                iyy="0.036694e-02"  iyz="0.000183e-02"
+                                                    izz="0.041529e-02" />
    </inertial>
       <visual>

Commit message: changed friction coefficients for stone_5 and stone_6 max_speed was changed to all the stones.

File: urdf_models/models/stone_1/urdf/stone_1.xacro (robot description, xacro)
@@ -13,5 +13,5 @@
 -->
 <robot name="stone_1" xmlns:xacro="http://ros.org/wiki/xacro">
-  <xacro:property name="mesh_file" value="package://urdf_models/models/stone_1/mesh/stone_1.stl" />
+  <xacro:property name="mesh_file" value="package://urdf_models/models/stone_1/mesh/stone_1.dae" />
   <xacro:property name="mass" value="1.0" />
   <link name="base_link"></link>
@@ -22,24 +22,24 @@
   </joint>
   <link name="base_link_inertia">
-  <inertial>
-    <mass value="${mass}" />  <!-- [kg] -->
-    <origin xyz="-0.0000142 0.0000139 0.0000031" />
-    <inertia ixx="0.008166e-02" ixy="-0.003668e-02" ixz="-0.000031e-02"
+     <inertial>
+    	<mass value="${mass}" />  <!-- [kg] -->
+    	<origin xyz="-0.0000142 0.0000139 0.0000031" />
+    	<inertia ixx="0.008166e-02" ixy="-0.003668e-02" ixz="-0.000031e-02"
                                 iyy="0.020183e-02"  iyz="0.000657e-02"
                                                     izz="0.024189e-02" />
-   </inertial>
-      <visual>
+   	 </inertial>
+  	 <visual>
         <origin xyz="0 0 0" rpy="0 0 0" />
         <geometry>
           <mesh filename="${mesh_file}" scale="1 1 1" />
         </geometry>
-      </visual>
-      <collision>
+   	</visual>
+   	<collision>
         <origin xyz="0 0 0" rpy="0 0 0" />
         <geometry>
           <mesh filename="${mesh_file}" scale="1 1 1" />
         </geometry>
-      </collision>
-    </link>
+  	</collision>
+  </link>
     <gazebo reference="base_link">
         <mu1 value="2.2"/>
@@ -51,10 +51,10 @@
             <surface>
               <bounce>
-                <restitution_coefficient> 0.1 </restitution_coefficient>
+                <restitution_coefficient> 0.0 </restitution_coefficient>
                 <threshold>0.</threshold>
               </bounce>
             <contact>
                 <ode>
-                  <max_vel>0.1</max_vel>
+                  <max_vel>10</max_vel>
                   <min_depth>0.001</min_depth>
                 </ode>
@@ -62,7 +62,4 @@
             </surface>
        </collision>
-        <material name="Gray">
-        <color rgba="0.8 0.8 0.8 1"/>
-      </material>
         <turnGravityOff>false</turnGravityOff>
     </gazebo>

File: urdf_models/models/stone_2/urdf/stone_2.xacro (robot description, xacro)
@@ -13,5 +13,5 @@
 -->
 <robot name="stone_2" xmlns:xacro="http://ros.org/wiki/xacro">
-  <xacro:property name="mesh_file" value="package://urdf_models/models/stone_2/mesh/stone_2.stl" />
+  <xacro:property name="mesh_file" value="package://urdf_models/models/stone_2/mesh/stone_2.dae" />
   <xacro:property name="mass" value="1.0" />
   <link name="base_link"></link>
@@ -52,16 +52,16 @@
       <fdir1 value="1 0 0"/>
       <collision>
-	        <surface>
+	      <surface>
 	          <bounce>
-	            <restitution_coefficient> 0.1 </restitution_coefficient>
+	            <restitution_coefficient> 0.0 </restitution_coefficient>
 	            <threshold>0.</threshold>
 	          </bounce>
-		      <contact>
+		        <contact>
 		          <ode>
-		            <max_vel>0.1</max_vel>
+		            <max_vel>10</max_vel>
 		            <min_depth>0.001</min_depth>
 		          </ode>
-		      </contact>
-	        </surface>
+		        </contact>
+	      </surface>
 	   </collision>
       <material name="Gray">

File: urdf_models/models/stone_3/urdf/stone_3.xacro (robot description, xacro)
@@ -54,5 +54,5 @@
 	        <surface>
 	          <bounce>
-	            <restitution_coefficient> 0.1 </restitution_coefficient>
+	            <restitution_coefficient> 10 </restitution_coefficient>
 	            <threshold>0.</threshold>
 	          </bounce>

File: urdf_models/models/stone_4/urdf/stone_4.xacro (robot description, xacro)
@@ -56,5 +56,5 @@
             <contact>
                 <ode>
-                  <max_vel>0.1</max_vel>
+                  <max_vel>10</max_vel>
                   <min_depth>0.001</min_depth>
                 </ode>

File: urdf_models/models/stone_5/urdf/stone_5.xacro (robot description, xacro)
@@ -43,5 +43,5 @@
     </link>
     <gazebo reference="base_link">
-        <mu1 value="2.2"/>
+        <mu1 value="0.5"/>
         <mu2 value="1.1"/>
         <kp  value="5000000.0" />
@@ -56,5 +56,5 @@
             <contact>
                 <ode>
-                  <max_vel>0.1</max_vel>
+                  <max_vel>10</max_vel>
                   <min_depth>0.001</min_depth>
                 </ode>

File: urdf_models/models/stone_6/urdf/stone_6.xacro (robot description, xacro)
@@ -43,5 +43,5 @@
     </link>
     <gazebo reference="base_link">
-        <mu1 value="2.2"/>
+        <mu1 value="0.5"/>
         <mu2 value="1.1"/>
         <kp  value="5000000.0" />
@@ -56,5 +56,5 @@
             <contact>
                 <ode>
-                  <max_vel>0.1</max_vel>
+                  <max_vel>10</max_vel>
                   <min_depth>0.001</min_depth>
                 </ode>

Commit message: Added stone formation.

File: urdf_models/models/stone_1/urdf/stone_1.xacro (robot description, xacro)
@@ -15,5 +15,13 @@
   <xacro:property name="mesh_file" value="package://urdf_models/models/stone_1/mesh/stone_1.dae" />
   <xacro:property name="mass" value="1.0" />
-  <link name="base_link"></link>
+  <link name="base_link">
+    <inertial>
+   	  <mass value="${mass}" />  <!-- [kg] -->
+   	  <origin xyz="-0.0000142 0.0000139 0.0000031" />
+   	  <inertia ixx="0.08166e-02" ixy="-0.03668e-02" ixz="-0.00031e-02"
+                                  iyy="0.20183e-02"  iyz="0.00657e-02"
+                                                      izz="0.24189e-02" />
+  	 </inertial>
+  </link>
   <joint name="base_joint" type="fixed">
     <origin xyz="0 0 0" rpy="0 0 0" />
@@ -22,11 +30,4 @@
   </joint>
   <link name="base_link_inertia">
-     <inertial>
-    	<mass value="${mass}" />  <!-- [kg] -->
-    	<origin xyz="-0.0000142 0.0000139 0.0000031" />
-    	<inertia ixx="0.008166e-02" ixy="-0.003668e-02" ixz="-0.000031e-02"
-                                iyy="0.020183e-02"  iyz="0.000657e-02"
-                                                    izz="0.024189e-02" />
-   	 </inertial>
   	 <visual>
         <origin xyz="0 0 0" rpy="0 0 0" />
@@ -42,25 +43,27 @@
   	</collision>
   </link>
-    <gazebo reference="base_link">
-        <mu1 value="0.1"/>
-        <mu2 value="0.1"/>
-        <kp  value="5000000.0" />
-        <kd  value="1.0" />
-        <fdir1 value="1 0 0"/>
-        <collision>
-            <surface>
-              <bounce>
-                <restitution_coefficient> 0.0 </restitution_coefficient>
-                <threshold>0.</threshold>
-              </bounce>
-            <contact>
-                <ode>
-                  <max_vel>10</max_vel>
-                  <min_depth>0.001</min_depth>
-                </ode>
-            </contact>
-            </surface>
-       </collision>
-        <turnGravityOff>false</turnGravityOff>
-    </gazebo>
+  <gazebo reference="base_link_inertia">
+    <mu1 value="0.1"/>
+    <mu2 value="0.1"/>
+    <kp  value="5000000.0" />
+    <kd  value="1.0" />
+    <fdir1 value="1 0 0"/>
+    <collision>
+    <surface>
+      <bounce>
+        <restitution_coefficient>0.1</restitution_coefficient>
+        <threshold>0.</threshold>
+      </bounce>
+      <contact>
+        <ode>
+          <max_vel>0</max_vel>
+          <min_depth>0.001</min_depth>
+        </ode>
+      </contact>
+    </surface>
+    </collision>
+    <material name="Gray">
+      <color rgba="0.8 0.8 0.8 1"/>
+    </material>
+  </gazebo>
 </robot>

Commit message: local adding of grasping set

File: urdf_models/models/stone_1/urdf/stone_1.xacro (robot description, xacro)
@@ -14,5 +14,5 @@
 <robot name="stone_1" xmlns:xacro="http://ros.org/wiki/xacro">
   <xacro:property name="mesh_file" value="package://urdf_models/models/stone_1/mesh/stone_1.dae" />
-  <xacro:property name="mass" value="1.0" />
+  <xacro:property name="mass" value="0.6" />
   <link name="base_link">
     <inertial>
@@ -22,5 +22,5 @@
                                   iyy="0.20183e-02"  iyz="0.00657e-02"
                                                       izz="0.24189e-02" />
-  	 </inertial>
+	 </inertial>
   </link>
   <joint name="base_joint" type="fixed">
@@ -44,6 +44,6 @@
   </link>
   <gazebo reference="base_link_inertia">
-    <mu1 value="0.1"/>
-    <mu2 value="0.1"/>
+    <mu1 value="10.0"/>
+    <mu2 value="10.0"/>
     <kp  value="5000000.0" />
     <kd  value="1.0" />

File: urdf_models/models/stone_3/urdf/stone_3.xacro (robot description, xacro)
@@ -46,6 +46,6 @@
   </link>
   <gazebo reference="base_link">
-    <mu1 value="0.1"/>
-    <mu2 value="0.1"/>
+    <mu1 value="100"/>
+    <mu2 value="100"/>
     <kp  value="5000000.0" />
     <kd  value="1.0" />
